Commit message: modify urdf file and fix some bugs

File: source/whole_body_tracking/whole_body_tracking/assets/roban_s22/urdf/biped_s17_hands.urdf (robot description, URDF)
Before this commit: robot biped_s17, 26 links, 25 joints
Links:
- added link zarm_l5_link, mass 1e-4; visual sphere radius=0.025
- added link zarm_r5_link, mass 1e-4; visual sphere radius=0.025
- link zarm_l4_link: geometry collision capsule length=0.03 radius=0.045; collision capsule length=0.08 radius=0.035
- link zarm_r4_link: geometry collision capsule length=0.03 radius=0.045; collision capsule length=0.08 radius=0.035
Joints:
- added joint zarm_l5_joint: type fixed, parent zarm_l4_link, child zarm_l5_link, origin xyz=0 0 -0.2085 rpy=0 0 0, axis 0 1 0, limit lower=-0.001 upper=0.001 effort=1 velocity=1.0
- added joint zarm_r5_joint: type fixed, parent zarm_r4_link, child zarm_r5_link, origin xyz=0 0 -0.2085 rpy=0 0 0, axis 0 1 0, limit lower=-0.001 upper=0.001 effort=1 velocity=1.0
