Commit message: fixed roban error

File: source/whole_body_tracking/whole_body_tracking/assets/roban_s22/urdf/biped_s17.urdf (robot description, URDF)
Before this commit: robot biped_s17, 26 links, 25 joints
Joints:
- joint zhead_1_joint: parent waist_yaw_link -> base_link

File: source/whole_body_tracking/whole_body_tracking/assets/unitree_description/urdf/g1/main.urdf (robot description, URDF)
Before this commit: robot g1, 40 links, 39 joints
Links:
- link head_link: geometry visual mesh filename=../../meshes/g1/head_link.STL
- link left_ankle_pitch_link: geometry visual mesh filename=../../meshes/g1/left_ankle_pitch_link.STL
- link left_ankle_roll_link: geometry collision cylinder length=0.05 radius=0.01; collision cylinder length=0.05 radius=0.01
- link left_elbow_link: geometry collision cylinder length=0.13 radius=0.035; visual mesh filename=../../meshes/g1/left_elbow_link.STL
- link left_hip_pitch_link: geometry visual mesh filename=../../meshes/g1/left_hip_pitch_link.STL
- link left_hip_roll_link: geometry collision cylinder length=0.2 radius=0.05; visual mesh filename=../../meshes/g1/left_hip_roll_link.STL
- link left_hip_yaw_link: geometry visual mesh filename=../../meshes/g1/left_hip_yaw_link.STL
- link left_knee_link: geometry collision cylinder length=0.2 radius=0.05; visual mesh filename=../../meshes/g1/left_knee_link.STL
- link left_rubber_hand: geometry visual mesh filename=../../meshes/g1/left_rubber_hand.STL
- link left_shoulder_pitch_link: geometry visual mesh filename=../../meshes/g1/left_shoulder_pitch_link.STL
- link left_shoulder_roll_link: geometry collision cylinder length=0.05 radius=0.035; visual mesh filename=../../meshes/g1/left_shoulder_roll_link.STL
- link left_shoulder_yaw_link: geometry collision cylinder length=0.13 radius=0.035; visual mesh filename=../../meshes/g1/left_shoulder_yaw_link.STL
- link left_wrist_pitch_link: geometry visual mesh filename=../../meshes/g1/left_wrist_pitch_link.STL
- link left_wrist_roll_link: geometry visual mesh filename=../../meshes/g1/left_wrist_roll_link.STL
- link left_wrist_yaw_link: geometry collision sphere radius=0.02; visual mesh filename=../../meshes/g1/left_wrist_yaw_link.STL
- link logo_link: geometry visual mesh filename=../../meshes/g1/logo_link.STL
- link pelvis: geometry collision sphere radius=0.07; visual mesh filename=../../meshes/g1/pelvis.STL
- link pelvis_contour_link: geometry visual mesh filename=../../meshes/g1/pelvis_contour_link.STL
- link right_ankle_pitch_link: geometry visual mesh filename=../../meshes/g1/right_ankle_pitch_link.STL
- link right_ankle_roll_link: geometry collision cylinder length=0.05 radius=0.01; collision cylinder length=0.05 radius=0.01
- link right_elbow_link: geometry collision cylinder length=0.13 radius=0.035; visual mesh filename=../../meshes/g1/right_elbow_link.STL
- link right_hip_pitch_link: geometry visual mesh filename=../../meshes/g1/right_hip_pitch_link.STL
- link right_hip_roll_link: geometry collision cylinder length=0.2 radius=0.05; visual mesh filename=../../meshes/g1/right_hip_roll_link.STL
- link right_hip_yaw_link: geometry visual mesh filename=../../meshes/g1/right_hip_yaw_link.STL
- link right_knee_link: geometry collision cylinder length=0.2 radius=0.05; visual mesh filename=../../meshes/g1/right_knee_link.STL
- link right_rubber_hand: geometry visual mesh filename=../../meshes/g1/right_rubber_hand.STL
- link right_shoulder_pitch_link: geometry visual mesh filename=../../meshes/g1/right_shoulder_pitch_link.STL
- link right_shoulder_roll_link: geometry collision cylinder length=0.05 radius=0.035; visual mesh filename=../../meshes/g1/right_shoulder_roll_link.STL
- link right_shoulder_yaw_link: geometry collision cylinder length=0.13 radius=0.035; visual mesh filename=../../meshes/g1/right_shoulder_yaw_link.STL
- link right_wrist_pitch_link: geometry visual mesh filename=../../meshes/g1/right_wrist_pitch_link.STL
- link right_wrist_roll_link: geometry visual mesh filename=../../meshes/g1/right_wrist_roll_link.STL
- link right_wrist_yaw_link: geometry collision sphere radius=0.02; visual mesh filename=../../meshes/g1/right_wrist_yaw_link.STL
- link torso_link: geometry collision cylinder length=0.01 radius=0.068; collision cylinder length=0.04 radius=0.065
- link waist_roll_link: geometry visual mesh filename=../../meshes/g1/waist_roll_link_rev_1_0.STL
- link waist_yaw_link: geometry visual mesh filename=../../meshes/g1/waist_yaw_link_rev_1_0.STL
