Commit message: add sim2sim

File: source/whole_body_tracking/whole_body_tracking/assets/unitree_description/urdf/g1/main.urdf (robot description, URDF)
Before this commit: robot g1, 40 links, 39 joints
Links:
- link pelvis: geometry collision sphere radius=0.05; visual mesh filename=../../meshes/g1/pelvis.STL
